Commit message: feat: complete robot control workflow
- unify app and firmware on the 16-byte protocol
- add teaching, servo calibration, and yaw PID
- document hardware, safety, and validation

File: simulator/models/robot_arm.urdf (robot description, URDF)
Before this commit: robot mobile_retrieval_arm, 8 links, 7 joints
Links:
- added link tcp_link, mass 0.000001
- link base_link: mass None -> 0.137140; geometry collision cylinder length=0.080 radius=0.055; visual mesh filename=base.stl scale=0.001 0.001 0.001
- link base_yaw_link: mass None -> 0.114160; geometry collision cylinder length=0.090 radius=0.047; visual mesh filename=central_shaft.stl scale=0.001 0.001 0.001
- link elbow_link: mass None -> 0.040770; geometry collision box size=0.114 0.034 0.045; visual mesh filename=servo_retainer.stl scale=0.001 0.001 0.001
- link gripper_finger_1_link: mass None -> 0.011850; geometry collision box size=0.064 0.016 0.016; visual mesh filename=bar_1.stl scale=0.001 0.001 0.001
- link gripper_finger_2_link: mass None -> 0.011610; geometry collision box size=0.064 0.016 0.016; visual mesh filename=bar_2.stl scale=0.001 0.001 0.001
- link shoulder_link: mass None -> 0.099100; geometry collision box size=0.038 0.026 0.135; visual mesh filename=forearm.stl scale=0.001 0.001 0.001
- link wrist_rotate_link: mass None -> 0.021440; geometry collision box size=0.078 0.036 0.036; visual mesh filename=gripper_base.stl scale=0.001 0.001 0.001
- link wrist_tilt_link: mass None -> 0.025150; geometry collision box size=0.095 0.044 0.042; visual mesh filename=gripper_cover.stl scale=0.001 0.001 0.001
Joints:
- added joint tcp_fixed_joint: type fixed, parent wrist_rotate_link, child tcp_link, origin xyz=0.125 0 0 rpy=0 0 0
- joint gripper_finger_1_joint: axis (none) -> 0 1 0; limit (none) -> lower=-0.18 upper=0.25 effort=0.08 velocity=3.0; type fixed -> revolute
- joint gripper_finger_2_joint: axis (none) -> 0 1 0; limit (none) -> lower=-0.25 upper=0.18 effort=0.08 velocity=3.0; type fixed -> revolute
